Commit message: goal checker for moveit_cpp_v3 added

File: tm_description/urdf/tm5-900-nominal.urdf (robot description, URDF)
Before this commit: robot tm5-900, 9 links, 8 joints
Links:
- added link gripper
Joints:
- added joint gripper_joint: type fixed, parent link_6, child gripper, origin xyz=0.000000 0.000000 0.215 rpy=0.000000 0.000000 0.000000

File: tm_description/urdf/tm5-900.urdf (robot description, URDF)
Before this commit: robot tm5-900, 9 links, 8 joints
Links:
- added link gripper
Joints:
- added joint gripper_joint: type fixed, parent link_6, child gripper, origin xyz=0.000000 0.000000 0.215 rpy=0.000000 0.000000 0.000000

File: tm_description/xacro/macro.tm5-900-nominal.urdf.xacro (robot description, xacro)
@@ -274,4 +274,10 @@
     <origin rpy="0.000000 0.000000 0.000000" xyz="0.000000 0.000000 0.000000" />
   </joint>
+  <link name="${prefix}gripper" />
+  <joint name="${prefix}gripper_joint" type="fixed">
+    <parent link="${prefix}link_6" />
+    <child link="${prefix}gripper" />
+    <origin rpy="0.000000 0.000000 0.000000" xyz="0.000000 0.000000 0.215" />
+  </joint>
 <!--LinkDescription-->
   </xacro:macro>

Commit message: goal checker for moveit_cpp_v4 added

File: tm_description/urdf/tm5-900-nominal.urdf (robot description, URDF)
Before this commit: robot tm5-900, 10 links, 9 joints
Joints:
- joint gripper_joint: origin xyz=0.000000 0.000000 0.215 rpy=0.000000 0.000000 0.000000 -> xyz=0.000000 0.000000 0.230 rpy=0.000000 0.000000 0.000000

File: tm_description/urdf/tm5-900.urdf (robot description, URDF)
Before this commit: robot tm5-900, 10 links, 9 joints
Joints:
- joint gripper_joint: origin xyz=0.000000 0.000000 0.215 rpy=0.000000 0.000000 0.000000 -> xyz=0.000000 0.000000 0.230 rpy=0.000000 0.000000 0.000000
