Commit message: moveir_cpp_v5

File: tm_description/urdf/tm5-900.urdf (robot description, URDF)
Before this commit: robot tm5-900, 10 links, 9 joints
Links:
- removed link gripper
Joints:
- removed joint gripper_joint

File: tm_description/xacro/macro.tm5-900-nominal-mod.urdf.xacro (robot description, xacro)
@@ -248,4 +248,5 @@
       <geometry>
         <!-- <mesh filename="package://tm_description/meshes/tm5-900/visual/tmr_ee.${format}" /> -->
+        <!-- <mesh filename="package://tm_description/meshes/tm5-900/visual/urdf_link6_modified.STL"/> -->
         <mesh filename="package://tm_description/meshes/tm5-900/visual/urdf_link6_modified_rg2less.STL"/>
       </geometry>
@@ -258,4 +259,5 @@
       <geometry>
         <!-- <mesh filename="package://tm_description/meshes/tm5-900/collision/tmr_ee_c.stl" /> -->
+        <!-- <mesh filename="package://tm_description/meshes/tm5-900/collision/urdf_link6_modified.STL"/> -->
         <mesh filename="package://tm_description/meshes/tm5-900/collision/urdf_link6_modified_rg2less.STL"/>
       </geometry>
@@ -294,7 +296,7 @@
   <xacro:include filename="$(find onrobot_rg_description)/urdf/onrobot_rg2_model.xacro" />
   <joint name="RG2_TM_attachment" type="fixed">
-    <parent link="flange" />  <!-- Adjust this to the actual last link of the TM5 arm -->
+    <parent link="flange" />
     <child link="onrobot_rg2_base_link" />
-    <origin xyz="0.0 0.0 0.0" rpy="0 0 1.5707" />  <!-- Adjust this to the correct position and orientation -->
+    <origin xyz="0.0 0.0 0.0" rpy="0 0 1.5707" />
   </joint>
   <!--LinkDescription-->
