Commit message: leaf boxes added separately

File: tm_description/xacro/macro.tm5-900-nominal-mod.urdf.xacro (robot description, xacro)
@@ -282,4 +282,10 @@
     <origin rpy="0.000000 0.000000 0.000000" xyz="0.000000 0.000000 0.230" />
   </joint>
+  <link name="${prefix}camera_link" />
+  <joint name="${prefix}camera_joint" type="fixed">
+    <parent link="${prefix}link_6" />
+    <child link="${prefix}camera_link" />
+    <origin rpy="0.000000 -1.5707 -1.5707" xyz="0.0175 0.1243 0.01933" />
+  </joint>
 <!--LinkDescription-->
   </xacro:macro>

Commit message: link_6 STL corrected

File: tm_description/xacro/macro.tm5-900-nominal-mod.urdf.xacro (robot description, xacro)
@@ -247,8 +247,11 @@
     <visual>
       <geometry>
-        <mesh filename="package://tm_description/meshes/tm5-900/visual/tmr_ee.${format}" />
-        <!-- <mesh filename="package://tm_description/meshes/tm5-900/visual/urdf_link6_modified.STL"/> -->
-      </geometry>
-      <material name="${color}" />
+        <!-- <mesh filename="package://tm_description/meshes/tm5-900/visual/tmr_ee.${format}" /> -->
+        <mesh filename="package://tm_description/meshes/tm5-900/visual/urdf_link6_modified.STL"/>
+      </geometry>
+      <material name="gray">
+          <color rgba="0.5 0.5 0.5 1.0"/>
+      </material>
+      <!-- <material name="${color}" /> -->
     </visual>
     <collision>

Commit message: RG2 Gripper included

File: tm_description/xacro/macro.tm5-900-nominal-mod.urdf.xacro (robot description, xacro)
@@ -248,5 +248,5 @@
       <geometry>
         <!-- <mesh filename="package://tm_description/meshes/tm5-900/visual/tmr_ee.${format}" /> -->
-        <mesh filename="package://tm_description/meshes/tm5-900/visual/urdf_link6_modified.STL"/>
+        <mesh filename="package://tm_description/meshes/tm5-900/visual/urdf_link6_modified_rg2less.STL"/>
       </geometry>
       <material name="gray">
@@ -258,5 +258,5 @@
       <geometry>
         <!-- <mesh filename="package://tm_description/meshes/tm5-900/collision/tmr_ee_c.stl" /> -->
-        <mesh filename="package://tm_description/meshes/tm5-900/collision/urdf_link6_modified.STL"/>
+        <mesh filename="package://tm_description/meshes/tm5-900/collision/urdf_link6_modified_rg2less.STL"/>
       </geometry>
     </collision>
@@ -291,5 +291,12 @@
     <origin rpy="0.000000 -1.5707 -1.5707" xyz="0.0175 0.1243 0.01933" />
   </joint>
-<!--LinkDescription-->
+  <!-- RG2 -->
+  <xacro:include filename="$(find onrobot_rg_description)/urdf/onrobot_rg2_model.xacro" />
+  <joint name="RG2_TM_attachment" type="fixed">
+    <parent link="flange" />  <!-- Adjust this to the actual last link of the TM5 arm -->
+    <child link="onrobot_rg2_base_link" />
+    <origin xyz="0.0 0.0 0.0" rpy="0 0 1.5707" />  <!-- Adjust this to the correct position and orientation -->
+  </joint>
+  <!--LinkDescription-->
   </xacro:macro>
 </robot>
